Commit message: update urdf

File: tiago_dual_absolute_meshes.urdf (robot description, URDF)
Before this commit: robot tiago_dual, 26 links, 25 joints
Links:
- link arm_left_1_link: geometry visual mesh filename=/home/jovyan/Multiverse/Multiverse-Resources/robots/pal_rob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 scale=1.0 1.0 1.0
- link arm_left_2_link: geometry visual mesh filename=/home/jovyan/Multiverse/Multiverse-Resources/robots/pal_rob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 scale=1.0 1.0 1.0
- link arm_left_3_link: geometry visual mesh filename=/home/jovyan/Multiverse/Multiverse-Resources/robots/pal_rob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 scale=1.0 1.0 1.0
- link arm_left_4_link: geometry visual mesh filename=/home/jovyan/Multiverse/Multiverse-Resources/robots/pal_rob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 scale=1.0 1.0 1.0
- link arm_left_5_link: geometry visual mesh filename=/home/jovyan/Multiverse/Multiverse-Resources/robots/pal_rob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 scale=1.0 1.0 1.0
- link arm_left_6_link: geometry visual mesh filename=/home/jovyan/Multiverse/Multiverse-Resources/robots/pal_rob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 scale=1.0 1.0 1.0
- link arm_left_7_link: geometry visual cylinder length=0.004999999888241291 radius=0.004999999888241291; visual cylinder length=0.009750000201165676 radius=0.02500000037252903
- link arm_right_1_link: geometry visual mesh filename=/home/jovyan/Multiverse/Multiverse-Resources/robots/pal_rob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 scale=1.0 1.0 1.0
- link arm_right_2_link: geometry visual mesh filename=/home/jovyan/Multiverse/Multiverse-Resources/robots/pal_rob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 scale=1.0 1.0 1.0
- link arm_right_3_link: geometry visual mesh filename=/home/jovyan/Multiverse/Multiverse-Resources/robots/pal_rob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 scale=1.0 1.0 1.0
- link arm_right_4_link: geometry visual mesh filename=/home/jovyan/Multiverse/Multiverse-Resources/robots/pal_rob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 scale=1.0 1.0 1.0
- link arm_right_5_link: geometry visual mesh filename=/home/jovyan/Multiverse/Multiverse-Resources/robots/pal_rob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 scale=1.0 1.0 1.0
- link arm_right_6_link: geometry visual mesh filename=/home/jovyan/Multiverse/Multiverse-Resources/robots/pal_rob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 scale=1.0 1.0 1.0
- link arm_right_7_link: geometry visual cylinder length=0.004999999888241291 radius=0.004999999888241291; visual cylinder length=0.009750000201165676 radius=0.02500000037252903
- link base_link: geometry visual box size=0.18000000715255737 0.20000000298023224 0.550000011920929; visual mesh filename=/home/jovyan/Multiverse/Multiverse-Resources/robots/pal_rob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 scale=1.0 1.0 1.0
- link gripper_left_left_finger_link: geometry visual mesh filename=/home/jovyan/Multiverse/Multiverse-Resources/robots/pal_rob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 scale=1.0 1.0 1.0
- link gripper_left_right_finger_link: geometry visual mesh filename=/home/jovyan/Multiverse/Multiverse-Resources/robots/pal_rob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 scale=1.0 1.0 1.0
- link gripper_right_left_finger_link: geometry visual mesh filename=/home/jovyan/Multiverse/Multiverse-Resources/robots/pal_rob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 scale=1.0 1.0 1.0
- link gripper_right_right_finger_link: geometry visual mesh filename=/home/jovyan/Multiverse/Multiverse-Resources/robots/pal_rob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 scale=1.0 1.0 1.0
- link head_1_link: geometry visual mesh filename=/home/jovyan/Multiverse/Multiverse-Resources/robots/pal_rob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 scale=1.0 1.0 1.0
- link head_2_link: geometry visual mesh filename=/home/jovyan/Multiverse/Multiverse-Resources/robots/pal_rob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 scale=1.0 1.0 1.0
- link torso_lift_link: geometry visual mesh filename=/home/jovyan/Multiverse/Multiverse-Resources/robots/pal_rob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 scale=1.0 1.0 1.0
- link wheel_front_left_link: geometry visual mesh filename=/home/jovyan/Multiverse/Multiverse-Resources/robots/pal_rob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 scale=1.0 1.0 1.0
- link wheel_front_right_link: geometry visual mesh filename=/home/jovyan/Multiverse/Multiverse-Resources/robots/pal_rob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 scale=1.0 1.0 1.0
- link wheel_rear_left_link: geometry visual mesh filename=/home/jovyan/Multiverse/Multiverse-Resources/robots/pal_rob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 scale=1.0 1.0 1.0
- link wheel_rear_right_link: geometry visual mesh filename=/home/jovyan/Multiverse/Multiverse-Resources/robots/pal_rob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 scale=1.0 1.0 1.0
