Commit message: update urdf

File: multiverse_configs/fera/ur5e.urdf (robot description, URDF)
Before this commit: robot ur, 14 links, 13 joints
Links:
- removed link base
- removed link base_link
- removed link base_link_inertia
- removed link flange
- removed link forearm_link
- removed link ft_frame
- removed link shoulder_link
- removed link tool0
- removed link tool1
- removed link upper_arm_link
- removed link world_robot
- removed link wrist_1_link
- removed link wrist_2_link
- removed link wrist_3_link
- added link gripper_tool_frame
- added link map
Joints:
- removed joint base_joint
- removed joint base_link-base_fixed_joint
- removed joint base_link-base_link_inertia
- removed joint elbow_joint
- removed joint flange-tool0
- removed joint flange-tool1
- removed joint shoulder_lift_joint
- removed joint shoulder_pan_joint
- removed joint wrist_1_joint
- removed joint wrist_2_joint
- removed joint wrist_3-flange
- removed joint wrist_3_joint
- removed joint wrist_3_link-ft_frame
- added joint gripper_tool_frame_joint: type fixed, parent robotiq_85_base_link, child gripper_tool_frame, origin xyz=0.0 0.0 0.144 rpy=0.0 0.0 0

Commit message: update urdf

File: multiverse_configs/fera/ur5e.urdf (robot description, URDF)
Before this commit: robot ur5e, 2 links, 1 joints
Links:
- added link base
- added link base_link
- added link base_link_inertia, mass 4.0; collision mesh filename=package://ur_description/meshes/ur5e/collision/base.stl; visual mesh filename=package://ur_description/meshes/ur5e/visual/base.dae
- added link flange
- added link forearm_link, mass 2.846; collision mesh filename=package://ur_description/meshes/ur5e/collision/forearm.stl; visual mesh filename=package://ur_description/meshes/ur5e/visual/forearm.dae
- added link ft_frame
- added link robotiq_85_base_link, mass 6.6320197e-01; collision mesh filename=package://robotiq_description/meshes/collision/2f_85/roboti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; visual mesh filename=package://robotiq_description/meshes/visual/2f_85/robotiq_b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
- added link robotiq_85_left_finger_link, mass 4.260376752e-02; collision mesh filename=package://robotiq_description/meshes/collision/2f_85/left_f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; visual mesh filename=package://robotiq_description/meshes/visual/2f_85/left_fing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
- added link robotiq_85_left_finger_tip_link, mass 4.268588744e-02; collision mesh filename=package://robotiq_description/meshes/collision/2f_85/left_f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; visual mesh filename=package://robotiq_description/meshes/visual/2f_85/left_fing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
- added link robotiq_85_left_inner_knuckle_link, mass 2.969376448e-02; collision mesh filename=package://robotiq_description/meshes/collision/2f_85/left_i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; visual mesh filename=package://robotiq_description/meshes/visual/2f_85/left_inne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
- added link robotiq_85_left_knuckle_link, mass 1.384773208e-02; collision mesh filename=package://robotiq_description/meshes/collision/2f_85/left_k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; visual mesh filename=package://robotiq_description/meshes/visual/2f_85/left_knuc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
- added link robotiq_85_right_finger_link, mass 4.260376752000000e-02; collision mesh filename=package://robotiq_description/meshes/collision/2f_85/right_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; visual mesh filename=package://robotiq_description/meshes/visual/2f_85/right_fin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
- added link robotiq_85_right_finger_tip_link, mass 4.268588744e-02; collision mesh filename=package://robotiq_description/meshes/collision/2f_85/right_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; visual mesh filename=package://robotiq_description/meshes/visual/2f_85/right_fin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
- added link robotiq_85_right_inner_knuckle_link, mass 2.969376448e-02; collision mesh filename=package://robotiq_description/meshes/collision/2f_85/right_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; visual mesh filename=package://robotiq_description/meshes/visual/2f_85/right_inn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
- added link robotiq_85_right_knuckle_link, mass 1.384773208e-02; collision mesh filename=package://robotiq_description/meshes/collision/2f_85/right_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; visual mesh filename=package://robotiq_description/meshes/visual/2f_85/right_knu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
- added link shoulder_link, mass 3.761; collision mesh filename=package://ur_description/meshes/ur5e/collision/shoulder.stl; visual mesh filename=package://ur_description/meshes/ur5e/visual/shoulder.dae
- added link tool0
- added link upper_arm_link, mass 8.058; collision mesh filename=package://ur_description/meshes/ur5e/collision/upperarm.stl; visual mesh filename=package://ur_description/meshes/ur5e/visual/upperarm.dae
- added link wrist_1_link, mass 1.37; collision mesh filename=package://ur_description/meshes/ur5e/collision/wrist1.stl; visual mesh filename=package://ur_description/meshes/ur5e/visual/wrist1.dae
- added link wrist_2_link, mass 1.3; collision mesh filename=package://ur_description/meshes/ur5e/collision/wrist2.stl; visual mesh filename=package://ur_description/meshes/ur5e/visual/wrist2.dae
- added link wrist_3_link, mass 0.365; collision mesh filename=package://ur_description/meshes/ur5e/collision/wrist3.stl; visual mesh filename=package://ur_description/meshes/ur5e/visual/wrist3.dae
Joints:
- added joint base_joint: type fixed, parent map, child base_link, origin xyz=0 0 0 rpy=0 0 0
- added joint base_link-base_fixed_joint: type fixed, parent base_link, child base, origin xyz=0 0 0 rpy=0 0 3.141592653589793
- added joint base_link-base_link_inertia: type fixed, parent base_link, child base_link_inertia, origin xyz=0 0 0 rpy=0 0 3.141592653589793
- added joint elbow_joint: type revolute, parent upper_arm_link, child forearm_link, origin xyz=-0.425 0 0 rpy=0 0 0, axis 0 0 1, limit lower=-3.141592653589793 upper=3.141592653589793 effort=150.0 velocity=3.141592653589793
- added joint flange-tool0: type fixed, parent flange, child tool0, origin xyz=0 0 0 rpy=1.5707963267948966 0 1.5707963267948966
- added joint robotiq_85_base_joint: type fixed, parent wrist_3_link, child robotiq_85_base_link, origin xyz=0.0 0.0 0.0 rpy=0.0 0.0 0.0
- added joint robotiq_85_left_finger_joint: type fixed, parent robotiq_85_left_knuckle_link, child robotiq_85_left_finger_link, origin xyz=0.03152616 0.0 -0.00376347 rpy=0 0 0
- added joint robotiq_85_left_finger_tip_joint: type revolute, parent robotiq_85_left_finger_link, child robotiq_85_left_finger_tip_link, origin xyz=0.00563134 0.0 0.04718515 rpy=0 0 0, axis 0 -1 0, limit lower=0.0 upper=0.8 effort=50 velocity=0.5, mimic joint=robotiq_85_left_knuckle_joint multiplier=-1
- added joint robotiq_85_left_inner_knuckle_joint: type revolute, parent robotiq_85_base_link, child robotiq_85_left_inner_knuckle_link, origin xyz=0.0127 0.0 0.06142 rpy=0 0 0, axis 0 -1 0, limit lower=0.0 upper=0.8 effort=50 velocity=0.5, mimic joint=robotiq_85_left_knuckle_joint
- added joint robotiq_85_left_knuckle_joint: type revolute, parent robotiq_85_base_link, child robotiq_85_left_knuckle_link, origin xyz=0.03060114 0.0 0.05490452 rpy=0 0 0, axis 0 -1 0, limit lower=0.0 upper=0.8 effort=50 velocity=0.5
- added joint robotiq_85_right_finger_joint: type fixed, parent robotiq_85_right_knuckle_link, child robotiq_85_right_finger_link, origin xyz=-0.03152616 0.0 -0.00376347 rpy=0 0 0
- added joint robotiq_85_right_finger_tip_joint: type revolute, parent robotiq_85_right_finger_link, child robotiq_85_right_finger_tip_link, origin xyz=-0.00563134 0.0 0.04718515 rpy=0 0 0, axis 0 -1 0, limit lower=0.0 upper=0.8 effort=50 velocity=0.5, mimic joint=robotiq_85_left_knuckle_joint
- added joint robotiq_85_right_inner_knuckle_joint: type revolute, parent robotiq_85_base_link, child robotiq_85_right_inner_knuckle_link, origin xyz=-0.0127 0.0 0.06142 rpy=0 0 0, axis 0 -1 0, limit lower=0.0 upper=0.8 effort=50 velocity=0.5, mimic joint=robotiq_85_left_knuckle_joint multiplier=-1
- added joint robotiq_85_right_knuckle_joint: type revolute, parent robotiq_85_base_link, child robotiq_85_right_knuckle_link, origin xyz=-0.03060114 0.0 0.05490452 rpy=0 0 0, axis 0 -1 0, limit lower=-0.8 upper=0.0 effort=50 velocity=0.5, mimic joint=robotiq_85_left_knuckle_joint multiplier=-1
- added joint shoulder_lift_joint: type revolute, parent shoulder_link, child upper_arm_link, origin xyz=0 0 0 rpy=1.570796327 0 0, axis 0 0 1, limit lower=-6.283185307179586 upper=6.283185307179586 effort=150.0 velocity=3.141592653589793
- added joint shoulder_pan_joint: type revolute, parent base_link_inertia, child shoulder_link, origin xyz=0 0 0.1625 rpy=0 0 0, axis 0 0 1, limit lower=-6.283185307179586 upper=6.283185307179586 effort=150.0 velocity=3.141592653589793
- added joint wrist_1_joint: type revolute, parent forearm_link, child wrist_1_link, origin xyz=-0.3922 0 0.1333 rpy=0 0 0, axis 0 0 1, limit lower=-6.283185307179586 upper=6.283185307179586 effort=28.0 velocity=3.141592653589793
- added joint wrist_2_joint: type revolute, parent wrist_1_link, child wrist_2_link, origin xyz=0 -0.0997 -2.044881182297852e-11 rpy=1.570796327 0 0, axis 0 0 1, limit lower=-6.283185307179586 upper=6.283185307179586 effort=28.0 velocity=3.141592653589793
- added joint wrist_3-flange: type fixed, parent wrist_3_link, child flange, origin xyz=0 0 0 rpy=0 -1.5707963267948966 -1.5707963267948966
- added joint wrist_3_joint: type revolute, parent wrist_2_link, child wrist_3_link, origin xyz=0 0.0996 -2.042830148012698e-11 rpy=1.570796326589793 3.141592653589793 3.141592653589793, axis 0 0 1, limit lower=-6.283185307179586 upper=6.283185307179586 effort=28.0 velocity=3.141592653589793
- added joint wrist_3_link-ft_frame: type fixed, parent wrist_3_link, child ft_frame, origin xyz=0 0 0 rpy=3.141592653589793 0 0
