Commit message: updated armar7 urdf

File: multiverse_configs/armar7/Armar7.urdf (robot description, URDF)
Before this commit: robot Armar7, 189 links, 188 joints
Links:
- link Ankle_body_link: geometry collision mesh filename=/home/repo/multiverse_configs/armar7/meshes/body_lower_leg.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 scale=1 1 1; visual mesh filename=/home/repo/multiverse_configs/armar7/meshes/body_lower_leg.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 scale=1 1 1
- link ArmL1_Cla1_body_link: geometry collision mesh filename=/home/repo/multiverse_configs/armar7/meshes/cla1_sho1_exo.s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 scale=1 1 1; visual mesh filename=/home/repo/multiverse_configs/armar7/meshes/cla1_sho1_exo.d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 scale=1 1 1
- link ArmL2_Sho1_body_link: geometry collision mesh filename=/home/repo/multiverse_configs/armar7/meshes/sho1_sho2_exo_u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 scale=1 1 1; visual mesh filename=/home/repo/multiverse_configs/armar7/meshes/sho1_sho2_exo.d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 scale=1 1 1
- link ArmL3_Sho2_body_link: geometry visual mesh filename=/home/repo/multiverse_configs/armar7/meshes/arm_sho2_ex.dae scale=1 1 1
- link ArmL4_Sho3_body_link: geometry collision mesh filename=/home/repo/multiverse_configs/armar7/meshes/left_arm_sho3.s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 scale=1 1 1; visual mesh filename=/home/repo/multiverse_configs/armar7/meshes/left_arm_sho3.d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 scale=1 1 1
- link ArmL5_Elb1_body_link: geometry collision mesh filename=/home/repo/multiverse_configs/armar7/meshes/elbow1_left.stl scale=1 1 1; visual mesh filename=/home/repo/multiverse_configs/armar7/meshes/elbow1_left.dae scale=1 1 1
- link ArmL6_Elb2_body_link: geometry collision mesh filename=/home/repo/multiverse_configs/armar7/meshes/wrist.stl scale=1 1 1; visual mesh filename=/home/repo/multiverse_configs/armar7/meshes/wrist.dae scale=1 1 1
- link ArmR1_Cla1_body_link: geometry collision mesh filename=/home/repo/multiverse_configs/armar7/meshes/cla1_sho1_exo.s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 scale=1 1 1; visual mesh filename=/home/repo/multiverse_configs/armar7/meshes/cla1_sho1_exo.d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 scale=1 1 1
- link ArmR2_Sho1_body_link: geometry collision mesh filename=/home/repo/multiverse_configs/armar7/meshes/sho1_sho2_exo_u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 scale=1 1 1; visual mesh filename=/home/repo/multiverse_configs/armar7/meshes/sho1_sho2_exo.d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 scale=1 1 1
- link ArmR3_Sho2_body_link: geometry visual mesh filename=/home/repo/multiverse_configs/armar7/meshes/arm_sho2_ex.dae scale=1 1 1
- link ArmR4_Sho3_body_link: geometry collision mesh filename=/home/repo/multiverse_configs/armar7/meshes/right_arm_sho3.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 scale=1 1 1; visual mesh filename=/home/repo/multiverse_configs/armar7/meshes/right_arm_sho3.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 scale=1 1 1
- link ArmR5_Elb1_body_link: geometry collision mesh filename=/home/repo/multiverse_configs/armar7/meshes/elbow1_right.stl scale=1 1 1; visual mesh filename=/home/repo/multiverse_configs/armar7/meshes/elbow1_right.dae scale=1 1 1
- link ArmR6_Elb2_body_link: geometry collision mesh filename=/home/repo/multiverse_configs/armar7/meshes/wrist.stl scale=1 1 1; visual mesh filename=/home/repo/multiverse_configs/armar7/meshes/wrist.dae scale=1 1 1
- link AzureKinect_body_link: geometry visual mesh filename=/home/repo/multiverse_configs/armar7/meshes/azure_kinect.dae scale=1 1 1
- link CenterArms_body_link: geometry collision mesh filename=/home/repo/multiverse_configs/armar7/meshes/armanbindung.stl scale=1 1 1; visual mesh filename=/home/repo/multiverse_configs/armar7/meshes/armanbindung.dae scale=1 1 1
- link Hand L Palm_link: geometry collision mesh filename=/home/repo/multiverse_configs/armar7/meshes/armar-7_palm_le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 scale=1 1 1; visual mesh filename=/home/repo/multiverse_configs/armar7/meshes/armar-7_palm_le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 scale=1 1 1
- link Hand R Palm_link: geometry collision mesh filename=/home/repo/multiverse_configs/armar7/meshes/armar-7_palm_ri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 scale=1 1 1; visual mesh filename=/home/repo/multiverse_configs/armar7/meshes/armar-7_palm_ri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 scale=1 1 1
- link HandL_Adapter_link: geometry visual mesh filename=/home/repo/multiverse_configs/armar7/meshes/handadapter.dae scale=1 1 1
- link HandR_Adapter_link: geometry visual mesh filename=/home/repo/multiverse_configs/armar7/meshes/handadapter.dae scale=1 1 1
- link Head_body_link: geometry collision mesh filename=/home/repo/multiverse_configs/armar7/meshes/head.stl scale=1 1 1; visual mesh filename=/home/repo/multiverse_configs/armar7/meshes/head.dae scale=1 1 1
- link Hip_body_link: geometry collision mesh filename=/home/repo/multiverse_configs/armar7/meshes/body_shoulder.s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 scale=1 1 1; visual mesh filename=/home/repo/multiverse_configs/armar7/meshes/body_shoulder.d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 scale=1 1 1
- link Index L 1 Body_link: geometry collision mesh filename=/home/repo/multiverse_configs/armar7/meshes/armar-7_index_p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 scale=1 1 1; visual mesh filename=/home/repo/multiverse_configs/armar7/meshes/armar-7_index_p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 scale=1 1 1
- link Index L 2 Body_link: geometry collision mesh filename=/home/repo/multiverse_configs/armar7/meshes/armar-7_index_i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 scale=1 1 1; visual mesh filename=/home/repo/multiverse_configs/armar7/meshes/armar-7_index_i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 scale=1 1 1
- link Index R 1 Body_link: geometry collision mesh filename=/home/repo/multiverse_configs/armar7/meshes/armar-7_index_p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 scale=1 1 1; visual mesh filename=/home/repo/multiverse_configs/armar7/meshes/armar-7_index_p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 scale=1 1 1
- link Index R 2 Body_link: geometry collision mesh filename=/home/repo/multiverse_configs/armar7/meshes/armar-7_index_i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 scale=1 1 1; visual mesh filename=/home/repo/multiverse_configs/armar7/meshes/armar-7_index_i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 scale=1 1 1
- link Knee_body_link: geometry collision mesh filename=/home/repo/multiverse_configs/armar7/meshes/thigh.stl scale=1 1 1; visual mesh filename=/home/repo/multiverse_configs/armar7/meshes/thigh.dae scale=1 1 1
- link LaserScannerBackLeftBody_link: geometry visual mesh filename=/home/repo/multiverse_configs/armar7/meshes/sick_tim_5xx.dae scale=1 1 1
- link LaserScannerBackRightBody_link: geometry visual mesh filename=/home/repo/multiverse_configs/armar7/meshes/sick_tim_5xx.dae scale=1 1 1
- link LaserScannerFrontBody_link: geometry visual mesh filename=/home/repo/multiverse_configs/armar7/meshes/sick_tim_5xx.dae scale=1 1 1
- link Middle L 1 Body_link: geometry collision mesh filename=/home/repo/multiverse_configs/armar7/meshes/armar-7_middle_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 scale=1 1 1; visual mesh filename=/home/repo/multiverse_configs/armar7/meshes/armar-7_middle_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 scale=1 1 1
- link Middle L 2 Body_link: geometry collision mesh filename=/home/repo/multiverse_configs/armar7/meshes/armar-7_middle_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 scale=1 1 1; visual mesh filename=/home/repo/multiverse_configs/armar7/meshes/armar-7_middle_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 scale=1 1 1
- link Middle R 1 Body_link: geometry collision mesh filename=/home/repo/multiverse_configs/armar7/meshes/armar-7_middle_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 scale=1 1 1; visual mesh filename=/home/repo/multiverse_configs/armar7/meshes/armar-7_middle_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 scale=1 1 1
- link Middle R 2 Body_link: geometry collision mesh filename=/home/repo/multiverse_configs/armar7/meshes/armar-7_middle_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 scale=1 1 1; visual mesh filename=/home/repo/multiverse_configs/armar7/meshes/armar-7_middle_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 scale=1 1 1
- link Neck_1_Yaw_body_link: geometry visual mesh filename=/home/repo/multiverse_configs/armar7/meshes/neck_yaw.dae scale=1 1 1
- link Neck_2_Pitch_body_link: geometry visual mesh filename=/home/repo/multiverse_configs/armar7/meshes/neck_pitch.dae scale=1 1 1
- link Neck_body_link: geometry collision mesh filename=/home/repo/multiverse_configs/armar7/meshes/neck.stl scale=1 1 1; visual mesh filename=/home/repo/multiverse_configs/armar7/meshes/neck.dae scale=1 1 1
- link Pinky L 1 Body_link: geometry collision mesh filename=/home/repo/multiverse_configs/armar7/meshes/armar-7_little_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 scale=1 1 1; visual mesh filename=/home/repo/multiverse_configs/armar7/meshes/armar-7_little_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 scale=1 1 1
- link Pinky L 2 Body_link: geometry collision mesh filename=/home/repo/multiverse_configs/armar7/meshes/armar-7_little_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 scale=1 1 1; visual mesh filename=/home/repo/multiverse_configs/armar7/meshes/armar-7_little_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 scale=1 1 1
- link Pinky R 1 Body_link: geometry collision mesh filename=/home/repo/multiverse_configs/armar7/meshes/armar-7_little_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 scale=1 1 1; visual mesh filename=/home/repo/multiverse_configs/armar7/meshes/armar-7_little_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 scale=1 1 1
- link Pinky R 2 Body_link: geometry collision mesh filename=/home/repo/multiverse_configs/armar7/meshes/armar-7_little_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 scale=1 1 1; visual mesh filename=/home/repo/multiverse_configs/armar7/meshes/armar-7_little_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 scale=1 1 1
- link Platform_body_link: geometry collision mesh filename=/home/repo/multiverse_configs/armar7/meshes/7a30000_plattfo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 scale=1 1 1; visual mesh filename=/home/repo/multiverse_configs/armar7/meshes/7a30000_plattfo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 scale=1 1 1
- link Ring L 1 Body_link: geometry collision mesh filename=/home/repo/multiverse_configs/armar7/meshes/armar-7_ring_pr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 scale=1 1 1; visual mesh filename=/home/repo/multiverse_configs/armar7/meshes/armar-7_ring_pr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 scale=1 1 1
- link Ring L 2 Body_link: geometry collision mesh filename=/home/repo/multiverse_configs/armar7/meshes/armar-7_ring_in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 scale=1 1 1; visual mesh filename=/home/repo/multiverse_configs/armar7/meshes/armar-7_ring_in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 scale=1 1 1
- link Ring R 1 Body_link: geometry collision mesh filename=/home/repo/multiverse_configs/armar7/meshes/armar-7_ring_pr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 scale=1 1 1; visual mesh filename=/home/repo/multiverse_configs/armar7/meshes/armar-7_ring_pr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 scale=1 1 1
- link Ring R 2 Body_link: geometry collision mesh filename=/home/repo/multiverse_configs/armar7/meshes/armar-7_ring_in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 scale=1 1 1; visual mesh filename=/home/repo/multiverse_configs/armar7/meshes/armar-7_ring_in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 scale=1 1 1
- link Thumb L 1 Body_link: geometry collision mesh filename=/home/repo/multiverse_configs/armar7/meshes/armar-7_thumb_b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 scale=1 1 1; visual mesh filename=/home/repo/multiverse_configs/armar7/meshes/armar-7_thumb_b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 scale=1 1 1
- link Thumb L 2 Body_link: geometry collision mesh filename=/home/repo/multiverse_configs/armar7/meshes/armar-7_thumb_p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 scale=1 1 1; visual mesh filename=/home/repo/multiverse_configs/armar7/meshes/armar-7_thumb_p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 scale=1 1 1
- link Thumb L 3 Body_link: geometry collision mesh filename=/home/repo/multiverse_configs/armar7/meshes/armar-7_thumb_d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 scale=1 1 1; visual mesh filename=/home/repo/multiverse_configs/armar7/meshes/armar-7_thumb_d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 scale=1 1 1
- link Thumb R 1 Body_link: geometry collision mesh filename=/home/repo/multiverse_configs/armar7/meshes/armar-7_thumb_b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 scale=1 1 1; visual mesh filename=/home/repo/multiverse_configs/armar7/meshes/armar-7_thumb_b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 scale=1 1 1
- link Thumb R 2 Body_link: geometry collision mesh filename=/home/repo/multiverse_configs/armar7/meshes/armar-7_thumb_p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 scale=1 1 1; visual mesh filename=/home/repo/multiverse_configs/armar7/meshes/armar-7_thumb_p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 scale=1 1 1
- link Thumb R 3 Body_link: geometry collision mesh filename=/home/repo/multiverse_configs/armar7/meshes/armar-7_thumb_d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 scale=1 1 1; visual mesh filename=/home/repo/multiverse_configs/armar7/meshes/armar-7_thumb_d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 scale=1 1 1
- link Torso_root_body_link: geometry collision mesh filename=/home/repo/multiverse_configs/armar7/meshes/ankle.stl scale=1 1 1; visual mesh filename=/home/repo/multiverse_configs/armar7/meshes/ankle.dae scale=1 1 1
