Commit message: updated velocity functionality

File: multiverse_configs/armar7/Armar7.urdf (robot description, URDF)
Before this commit: robot Armar7, 189 links, 188 joints
Joints:
- joint Ankle: limit lower=-0.757037 upper=0 effort=-1 velocity=-1 -> lower=-0.757037 upper=0 effort=-1 velocity=1.0
- joint Ankle_body: limit lower=0 upper=0 effort=-1 velocity=-1 -> lower=0 upper=0 effort=-1 velocity=1
- joint Ankle_ref: limit lower=0 upper=0 effort=-1 velocity=-1 -> lower=0 upper=0 effort=-1 velocity=1
- joint ArmL1_Cla1: limit lower=-1.41372 upper=1.41372 effort=-1 velocity=-1 -> lower=-1.41372 upper=1.41372 effort=-1 velocity=1
- joint ArmL1_Cla1_body: limit lower=0 upper=0 effort=-1 velocity=-1 -> lower=0 upper=0 effort=-1 velocity=1
- joint ArmL1_Cla1_link: limit lower=0 upper=0 effort=-1 velocity=-1 -> lower=0 upper=0 effort=-1 velocity=1
- joint ArmL2_Sho1: limit lower=-3.14159 upper=3.14159 effort=-1 velocity=-1 -> lower=-3.14159 upper=3.14159 effort=-1 velocity=1
- joint ArmL2_Sho1_body: limit lower=0 upper=0 effort=-1 velocity=-1 -> lower=0 upper=0 effort=-1 velocity=1
- joint ArmL2_Sho1_link: limit lower=0 upper=0 effort=-1 velocity=-1 -> lower=0 upper=0 effort=-1 velocity=1
- joint ArmL3_Sho2: limit lower=0.0872665 upper=3.24631 effort=-1 velocity=-1 -> lower=0.0872665 upper=3.24631 effort=-1 velocity=1
- joint ArmL3_Sho2_body: limit lower=0 upper=0 effort=-1 velocity=-1 -> lower=0 upper=0 effort=-1 velocity=1
- joint ArmL3_Sho2_link: limit lower=0 upper=0 effort=-1 velocity=-1 -> lower=0 upper=0 effort=-1 velocity=1
- joint ArmL4_Sho3: limit lower=-3.14159 upper=3.14159 effort=-1 velocity=-1 -> lower=-3.14159 upper=3.14159 effort=-1 velocity=1
- joint ArmL4_Sho3_body: limit lower=0 upper=0 effort=-1 velocity=-1 -> lower=0 upper=0 effort=-1 velocity=1
- joint ArmL5_Elb1: limit lower=0 upper=2.37365 effort=-1 velocity=-1 -> lower=0 upper=2.37365 effort=-1 velocity=1
- joint ArmL5_Elb1_body: limit lower=0 upper=0 effort=-1 velocity=-1 -> lower=0 upper=0 effort=-1 velocity=1
- joint ArmL5_Elb_link: limit lower=0 upper=0 effort=-1 velocity=-1 -> lower=0 upper=0 effort=-1 velocity=1
- joint ArmL6_Elb2: limit lower=-3.14159 upper=3.14159 effort=-1 velocity=-1 -> lower=-3.14159 upper=3.14159 effort=-1 velocity=1
- joint ArmL6_Elb2_body: limit lower=0 upper=0 effort=-1 velocity=-1 -> lower=0 upper=0 effort=-1 velocity=1
- joint ArmL7_Wri_link: limit lower=0 upper=0 effort=-1 velocity=-1 -> lower=0 upper=0 effort=-1 velocity=1
- joint ArmL7_Wrist_Hemisphere_A: limit lower=-0.541052 upper=0.680678 effort=-1 velocity=-1 -> lower=-0.541052 upper=0.680678 effort=-1 velocity=1
- joint ArmL8_Wrist_Hemisphere_B: limit lower=-0.541052 upper=0.680678 effort=-1 velocity=-1 -> lower=-0.541052 upper=0.680678 effort=-1 velocity=1
- joint ArmL_Wrist_Mechanism_Center: limit lower=0 upper=0 effort=-1 velocity=-1 -> lower=0 upper=0 effort=-1 velocity=1
- joint ArmR1_Cla1: limit lower=-1.41372 upper=1.41372 effort=-1 velocity=-1 -> lower=-1.41372 upper=1.41372 effort=-1 velocity=1
- joint ArmR1_Cla1_body: limit lower=0 upper=0 effort=-1 velocity=-1 -> lower=0 upper=0 effort=-1 velocity=1
- joint ArmR1_Cla1_link: limit lower=0 upper=0 effort=-1 velocity=-1 -> lower=0 upper=0 effort=-1 velocity=1
- joint ArmR2_Sho1: limit lower=-3.14159 upper=3.14159 effort=-1 velocity=-1 -> lower=-3.14159 upper=3.14159 effort=-1 velocity=1
- joint ArmR2_Sho1_body: limit lower=0 upper=0 effort=-1 velocity=-1 -> lower=0 upper=0 effort=-1 velocity=1
- joint ArmR3_Sho2: limit lower=0.0872665 upper=3.24631 effort=-1 velocity=-1 -> lower=0.0872665 upper=3.24631 effort=-1 velocity=1
- joint ArmR3_Sho2_body: limit lower=0 upper=0 effort=-1 velocity=-1 -> lower=0 upper=0 effort=-1 velocity=1
- joint ArmR3_Sho2_link: limit lower=0 upper=0 effort=-1 velocity=-1 -> lower=0 upper=0 effort=-1 velocity=1
- joint ArmR4_Sho3: limit lower=-3.14159 upper=3.14159 effort=-1 velocity=-1 -> lower=-3.14159 upper=3.14159 effort=-1 velocity=1
- joint ArmR4_Sho3_body: limit lower=0 upper=0 effort=-1 velocity=-1 -> lower=0 upper=0 effort=-1 velocity=1
- joint ArmR5_Elb1: limit lower=0 upper=2.37365 effort=-1 velocity=-1 -> lower=0 upper=2.37365 effort=-1 velocity=1
- joint ArmR5_Elb1_body: limit lower=0 upper=0 effort=-1 velocity=-1 -> lower=0 upper=0 effort=-1 velocity=1
- joint ArmR5_Elb_link: limit lower=0 upper=0 effort=-1 velocity=-1 -> lower=0 upper=0 effort=-1 velocity=1
- joint ArmR6_Elb2: limit lower=-3.14159 upper=3.14159 effort=-1 velocity=-1 -> lower=-3.14159 upper=3.14159 effort=-1 velocity=1
- joint ArmR6_Elb2_body: limit lower=0 upper=0 effort=-1 velocity=-1 -> lower=0 upper=0 effort=-1 velocity=1
- joint ArmR7_Wri_link: limit lower=0 upper=0 effort=-1 velocity=-1 -> lower=0 upper=0 effort=-1 velocity=1
- joint ArmR7_Wrist_Hemisphere_A: limit lower=-0.541052 upper=0.680678 effort=-1 velocity=-1 -> lower=-0.541052 upper=0.680678 effort=-1 velocity=1
- joint ArmR8_Wrist_Hemisphere_B: limit lower=-0.541052 upper=0.680678 effort=-1 velocity=-1 -> lower=-0.541052 upper=0.680678 effort=-1 velocity=1
- joint ArmR_Sho_link: limit lower=0 upper=0 effort=-1 velocity=-1 -> lower=0 upper=0 effort=-1 velocity=1
- joint ArmR_Wrist_Mechanism_Center: limit lower=0 upper=0 effort=-1 velocity=-1 -> lower=0 upper=0 effort=-1 velocity=1
- joint AzureKinect: limit lower=0 upper=0 effort=-1 velocity=-1 -> lower=0 upper=0 effort=-1 velocity=1
- joint AzureKinect_Base: limit lower=0 upper=0 effort=-1 velocity=-1 -> lower=0 upper=0 effort=-1 velocity=1
- joint AzureKinect_Calibration: limit lower=0 upper=0 effort=-1 velocity=-1 -> lower=0 upper=0 effort=-1 velocity=1
- joint AzureKinect_Depth: limit lower=0 upper=0 effort=-1 velocity=-1 -> lower=0 upper=0 effort=-1 velocity=1
- joint AzureKinect_RGB: limit lower=0 upper=0 effort=-1 velocity=-1 -> lower=0 upper=0 effort=-1 velocity=1
- joint AzureKinect_body: limit lower=0 upper=0 effort=-1 velocity=-1 -> lower=0 upper=0 effort=-1 velocity=1
- joint CenterArms_body: limit lower=0 upper=0 effort=-1 velocity=-1 -> lower=0 upper=0 effort=-1 velocity=1
- joint CenterArms_link: limit lower=0 upper=0 effort=-1 velocity=-1 -> lower=0 upper=0 effort=-1 velocity=1
- joint DepthCameraSim: limit lower=0 upper=0 effort=-1 velocity=-1 -> lower=0 upper=0 effort=-1 velocity=1
- joint Dummy_Platform: limit lower=0 upper=0 effort=-1 velocity=-1 -> lower=0 upper=0 effort=-1 velocity=1
- joint FT L Root: limit lower=0 upper=0 effort=-1 velocity=-1 -> lower=0 upper=0 effort=-1 velocity=1
- joint FT R Root: limit lower=0 upper=0 effort=-1 velocity=-1 -> lower=0 upper=0 effort=-1 velocity=1
- joint Gaze_Root: limit lower=0 upper=0 effort=-1 velocity=-1 -> lower=0 upper=0 effort=-1 velocity=1
- joint Hand L Col: limit lower=0 upper=0 effort=-1 velocity=-1 -> lower=0 upper=0 effort=-1 velocity=1
- joint Hand L GCP: limit lower=0 upper=0 effort=-1 velocity=-1 -> lower=0 upper=0 effort=-1 velocity=1
- joint Hand L Index TCP: limit lower=0 upper=0 effort=-1 velocity=-1 -> lower=0 upper=0 effort=-1 velocity=1
- joint Hand L Palm: limit lower=0 upper=0 effort=-1 velocity=-1 -> lower=0 upper=0 effort=-1 velocity=1
- joint Hand L Power TCP: limit lower=0 upper=0 effort=-1 velocity=-1 -> lower=0 upper=0 effort=-1 velocity=1
- joint Hand L Precision TCP: limit lower=0 upper=0 effort=-1 velocity=-1 -> lower=0 upper=0 effort=-1 velocity=1
- joint Hand L Root: limit lower=0 upper=0 effort=-1 velocity=-1 -> lower=0 upper=0 effort=-1 velocity=1
- joint Hand L TCP: limit lower=0 upper=0 effort=-1 velocity=-1 -> lower=0 upper=0 effort=-1 velocity=1
- joint Hand R Col: limit lower=0 upper=0 effort=-1 velocity=-1 -> lower=0 upper=0 effort=-1 velocity=1
- joint Hand R GCP: limit lower=0 upper=0 effort=-1 velocity=-1 -> lower=0 upper=0 effort=-1 velocity=1
- joint Hand R Index TCP: limit lower=0 upper=0 effort=-1 velocity=-1 -> lower=0 upper=0 effort=-1 velocity=1
- joint Hand R Palm: limit lower=0 upper=0 effort=-1 velocity=-1 -> lower=0 upper=0 effort=-1 velocity=1
- joint Hand R Power TCP: limit lower=0 upper=0 effort=-1 velocity=-1 -> lower=0 upper=0 effort=-1 velocity=1
- joint Hand R Precision TCP: limit lower=0 upper=0 effort=-1 velocity=-1 -> lower=0 upper=0 effort=-1 velocity=1
- joint Hand R Root: limit lower=0 upper=0 effort=-1 velocity=-1 -> lower=0 upper=0 effort=-1 velocity=1
- joint Hand R TCP: limit lower=0 upper=0 effort=-1 velocity=-1 -> lower=0 upper=0 effort=-1 velocity=1
- joint HandL_Adapter: limit lower=0 upper=0 effort=-1 velocity=-1 -> lower=0 upper=0 effort=-1 velocity=1
- joint HandL_Base: limit lower=0 upper=0 effort=-1 velocity=-1 -> lower=0 upper=0 effort=-1 velocity=1
- joint HandR_Adapter: limit lower=0 upper=0 effort=-1 velocity=-1 -> lower=0 upper=0 effort=-1 velocity=1
- joint HandR_Base: limit lower=0 upper=0 effort=-1 velocity=-1 -> lower=0 upper=0 effort=-1 velocity=1
- joint Head_Root: limit lower=0 upper=0 effort=-1 velocity=-1 -> lower=0 upper=0 effort=-1 velocity=1
- joint Head_body: limit lower=0 upper=0 effort=-1 velocity=-1 -> lower=0 upper=0 effort=-1 velocity=1
- joint Hip: limit lower=0 upper=2.18166 effort=-1 velocity=-1 -> lower=0 upper=2.18166 effort=-1 velocity=1.0
- joint Hip_body: limit lower=0 upper=0 effort=-1 velocity=-1 -> lower=0 upper=0 effort=-1 velocity=1
- joint Hip_body_monitor: limit lower=0 upper=0 effort=-1 velocity=-1 -> lower=0 upper=0 effort=-1 velocity=1
- joint Hip_body_prim: limit lower=0 upper=0 effort=-1 velocity=-1 -> lower=0 upper=0 effort=-1 velocity=1
- joint Hip_link: limit lower=0 upper=0 effort=-1 velocity=-1 -> lower=0 upper=0 effort=-1 velocity=1
- joint Index L 1 Body: limit lower=0 upper=0 effort=-1 velocity=-1 -> lower=0 upper=0 effort=-1 velocity=1
- joint Index L 2 Body: limit lower=0 upper=0 effort=-1 velocity=-1 -> lower=0 upper=0 effort=-1 velocity=1
- joint Index L Tip: limit lower=0 upper=0 effort=-1 velocity=-1 -> lower=0 upper=0 effort=-1 velocity=1
- joint Index R 1 Body: limit lower=0 upper=0 effort=-1 velocity=-1 -> lower=0 upper=0 effort=-1 velocity=1
- joint Index R 2 Body: limit lower=0 upper=0 effort=-1 velocity=-1 -> lower=0 upper=0 effort=-1 velocity=1
- joint Index R Tip: limit lower=0 upper=0 effort=-1 velocity=-1 -> lower=0 upper=0 effort=-1 velocity=1
- joint Knee: limit lower=0 upper=1.74533 effort=-1 velocity=-1 -> lower=0 upper=1.74533 effort=-1 velocity=1.0
- joint Knee_body: limit lower=0 upper=0 effort=-1 velocity=-1 -> lower=0 upper=0 effort=-1 velocity=1
- joint Knee_body_prim: limit lower=0 upper=0 effort=-1 velocity=-1 -> lower=0 upper=0 effort=-1 velocity=1
- joint Knee_body_ref: limit lower=0 upper=0 effort=-1 velocity=-1 -> lower=0 upper=0 effort=-1 velocity=1
- joint Knee_link: limit lower=0 upper=0 effort=-1 velocity=-1 -> lower=0 upper=0 effort=-1 velocity=1
- joint LaserScannerBackLeft: limit lower=0 upper=0 effort=-1 velocity=-1 -> lower=0 upper=0 effort=-1 velocity=1
- joint LaserScannerBackLeftBody: limit lower=0 upper=0 effort=-1 velocity=-1 -> lower=0 upper=0 effort=-1 velocity=1
- joint LaserScannerBackRight: limit lower=0 upper=0 effort=-1 velocity=-1 -> lower=0 upper=0 effort=-1 velocity=1
- joint LaserScannerBackRightBody: limit lower=0 upper=0 effort=-1 velocity=-1 -> lower=0 upper=0 effort=-1 velocity=1
- joint LaserScannerFront: limit lower=0 upper=0 effort=-1 velocity=-1 -> lower=0 upper=0 effort=-1 velocity=1
- joint LaserScannerFrontBody: limit lower=0 upper=0 effort=-1 velocity=-1 -> lower=0 upper=0 effort=-1 velocity=1
- joint Middle L 1 Body: limit lower=0 upper=0 effort=-1 velocity=-1 -> lower=0 upper=0 effort=-1 velocity=1
- joint Middle L 2 Body: limit lower=0 upper=0 effort=-1 velocity=-1 -> lower=0 upper=0 effort=-1 velocity=1
- joint Middle L Tip: limit lower=0 upper=0 effort=-1 velocity=-1 -> lower=0 upper=0 effort=-1 velocity=1
- joint Middle R 1 Body: limit lower=0 upper=0 effort=-1 velocity=-1 -> lower=0 upper=0 effort=-1 velocity=1
- joint Middle R 2 Body: limit lower=0 upper=0 effort=-1 velocity=-1 -> lower=0 upper=0 effort=-1 velocity=1
- joint Middle R Tip: limit lower=0 upper=0 effort=-1 velocity=-1 -> lower=0 upper=0 effort=-1 velocity=1
- joint Neck_1_Yaw_body: limit lower=0 upper=0 effort=-1 velocity=-1 -> lower=0 upper=0 effort=-1 velocity=1
- joint Neck_2_Pitch_body: limit lower=0 upper=0 effort=-1 velocity=-1 -> lower=0 upper=0 effort=-1 velocity=1
- joint Neck_Root: limit lower=0 upper=0 effort=-1 velocity=-1 -> lower=0 upper=0 effort=-1 velocity=1
- joint Neck_body: limit lower=0 upper=0 effort=-1 velocity=-1 -> lower=0 upper=0 effort=-1 velocity=1
- joint OmniWheelBack: limit lower=0 upper=0 effort=-1 velocity=-1 -> lower=0 upper=0 effort=-1 velocity=1
- joint OmniWheelBackGroundContact: limit lower=0 upper=0 effort=-1 velocity=-1 -> lower=0 upper=0 effort=-1 velocity=1
- joint OmniWheelFrontLeft: limit lower=0 upper=0 effort=-1 velocity=-1 -> lower=0 upper=0 effort=-1 velocity=1
- joint OmniWheelFrontLeftGroundContact: limit lower=0 upper=0 effort=-1 velocity=-1 -> lower=0 upper=0 effort=-1 velocity=1
- joint OmniWheelFrontRight: limit lower=0 upper=0 effort=-1 velocity=-1 -> lower=0 upper=0 effort=-1 velocity=1
- joint OmniWheelFrontRightGroundContact: limit lower=0 upper=0 effort=-1 velocity=-1 -> lower=0 upper=0 effort=-1 velocity=1
- joint Pinky L 1 Body: limit lower=0 upper=0 effort=-1 velocity=-1 -> lower=0 upper=0 effort=-1 velocity=1
- joint Pinky L 2 Body: limit lower=0 upper=0 effort=-1 velocity=-1 -> lower=0 upper=0 effort=-1 velocity=1
- joint Pinky L Tip: limit lower=0 upper=0 effort=-1 velocity=-1 -> lower=0 upper=0 effort=-1 velocity=1
- joint Pinky R 1 Body: limit lower=0 upper=0 effort=-1 velocity=-1 -> lower=0 upper=0 effort=-1 velocity=1
- joint Pinky R 2 Body: limit lower=0 upper=0 effort=-1 velocity=-1 -> lower=0 upper=0 effort=-1 velocity=1
- joint Pinky R Tip: limit lower=0 upper=0 effort=-1 velocity=-1 -> lower=0 upper=0 effort=-1 velocity=1
- joint Platform: limit lower=0 upper=0 effort=-1 velocity=-1 -> lower=0 upper=0 effort=-1 velocity=1
- joint Platform-navigation-colmodel: limit lower=0 upper=0 effort=-1 velocity=-1 -> lower=0 upper=0 effort=-1 velocity=1
- joint Platform_body: limit lower=0 upper=0 effort=-1 velocity=-1 -> lower=0 upper=0 effort=-1 velocity=1
- joint Ring L 1 Body: limit lower=0 upper=0 effort=-1 velocity=-1 -> lower=0 upper=0 effort=-1 velocity=1
- joint Ring L 2 Body: limit lower=0 upper=0 effort=-1 velocity=-1 -> lower=0 upper=0 effort=-1 velocity=1
- joint Ring L Tip: limit lower=0 upper=0 effort=-1 velocity=-1 -> lower=0 upper=0 effort=-1 velocity=1
- joint Ring R 1 Body: limit lower=0 upper=0 effort=-1 velocity=-1 -> lower=0 upper=0 effort=-1 velocity=1
- joint Ring R 2 Body: limit lower=0 upper=0 effort=-1 velocity=-1 -> lower=0 upper=0 effort=-1 velocity=1
- joint Ring R Tip: limit lower=0 upper=0 effort=-1 velocity=-1 -> lower=0 upper=0 effort=-1 velocity=1
- joint Stereo_Base: limit lower=0 upper=0 effort=-1 velocity=-1 -> lower=0 upper=0 effort=-1 velocity=1
- joint Stereo_Calib: limit lower=0 upper=0 effort=-1 velocity=-1 -> lower=0 upper=0 effort=-1 velocity=1
- joint Stereo_Left: limit lower=0 upper=0 effort=-1 velocity=-1 -> lower=0 upper=0 effort=-1 velocity=1
- joint Stereo_Right: limit lower=0 upper=0 effort=-1 velocity=-1 -> lower=0 upper=0 effort=-1 velocity=1
- joint Stereo_SensorPlane: limit lower=0 upper=0 effort=-1 velocity=-1 -> lower=0 upper=0 effort=-1 velocity=1
- joint Thumb L 1 Body: limit lower=0 upper=0 effort=-1 velocity=-1 -> lower=0 upper=0 effort=-1 velocity=1
- joint Thumb L 2 Body: limit lower=0 upper=0 effort=-1 velocity=-1 -> lower=0 upper=0 effort=-1 velocity=1
- joint Thumb L 3 Body: limit lower=0 upper=0 effort=-1 velocity=-1 -> lower=0 upper=0 effort=-1 velocity=1
- joint Thumb L Tip: limit lower=0 upper=0 effort=-1 velocity=-1 -> lower=0 upper=0 effort=-1 velocity=1
- joint Thumb R 1 Body: limit lower=0 upper=0 effort=-1 velocity=-1 -> lower=0 upper=0 effort=-1 velocity=1
- joint Thumb R 2 Body: limit lower=0 upper=0 effort=-1 velocity=-1 -> lower=0 upper=0 effort=-1 velocity=1
- joint Thumb R 3 Body: limit lower=0 upper=0 effort=-1 velocity=-1 -> lower=0 upper=0 effort=-1 velocity=1
- joint Thumb R Tip: limit lower=0 upper=0 effort=-1 velocity=-1 -> lower=0 upper=0 effort=-1 velocity=1
- joint ToF L Palm: limit lower=0 upper=0 effort=-1 velocity=-1 -> lower=0 upper=0 effort=-1 velocity=1
- joint ToF R Palm: limit lower=0 upper=0 effort=-1 velocity=-1 -> lower=0 upper=0 effort=-1 velocity=1
- joint Torso_link: limit lower=0 upper=0 effort=-1 velocity=-1 -> lower=0 upper=0 effort=-1 velocity=1
- joint Torso_mount: limit lower=0 upper=0 effort=-1 velocity=-1 -> lower=0 upper=0 effort=-1 velocity=1
- joint Torso_root_body: limit lower=0 upper=0 effort=-1 velocity=-1 -> lower=0 upper=0 effort=-1 velocity=1
- joint Torso_root_link: limit lower=0 upper=0 effort=-1 velocity=-1 -> lower=0 upper=0 effort=-1 velocity=1
- joint UpperBody_body: limit lower=0 upper=0 effort=-1 velocity=-1 -> lower=0 upper=0 effort=-1 velocity=1
- joint X_Platform: limit lower=-10 upper=10 effort=-1 velocity=-1 -> lower=-10 upper=10 effort=-1 velocity=1
- joint Y_Platform: limit lower=-10 upper=10 effort=-1 velocity=-1 -> lower=-10 upper=10 effort=-1 velocity=1
